File: HARDWARE/quizbuzzer/quizbuzzer.sch (KiCad schematic (older format))
At the start: 73 parts, among them J1 Bulb1, J10 Reciver 1, J11 Reciver 2, J12 Reciver 3, J13 Reciver 4, J14 Reciver 5, J15 Reciver 6, J16 Reciver 7, J17 Reciver 8, J18 Powerjack, J19 MP3out, J2 Bulb2, J20 I2C, J3 Bulb3, J4 Bulb4, J5 Bulb5, J6 Bulb6, J7 Bulb7, J8 Bulb8, J9 Controls, K1 SANYOU_SRD_Form_A, K2 SANYOU_SRD_Form_A, K3 SANYOU_SRD_Form_A, K4 SANYOU_SRD_Form_A, K5 SANYOU_SRD_Form_A, K6 SANYOU_SRD_Form_A, K7 SANYOU_SRD_Form_A, K8 SANYOU_SRD_Form_A, Q1 2N3904, Q2 2N3904, Q3 2N3904, Q4 2N3904, Q5 2N3904, Q6 2N3904, Q7 2N3904, Q8 2N3904, U1 74HC4051, U2 74HC4051, U3 L7805

Commit message: V0.1.0 sent to printer
Parts:
- removed D1, D2, D3, D4, D5, D6, D7, D8: 1N4007, Diode_THT:D_DO-41_SOD81_P10.16mm_Horizontal, symbol Diode:1N4007
- removed D10, D11, D12, D13, D14, D15, D16, D9: LED, LED_THT:LED_D5.0mm, symbol Device:LED
- removed J1: Bulb1, Connector_Molex:Molex_KK-254_AE-6410-02A_1x02_P2.54mm_Vertical, symbol Connector:Conn_01x02_Female
- removed J2: Bulb2, Connector_Molex:Molex_KK-254_AE-6410-02A_1x02_P2.54mm_Vertical, symbol Connector:Conn_01x02_Female
- removed J3: Bulb3, Connector_Molex:Molex_KK-254_AE-6410-02A_1x02_P2.54mm_Vertical, symbol Connector:Conn_01x02_Female
- removed J4: Bulb4, Connector_Molex:Molex_KK-254_AE-6410-02A_1x02_P2.54mm_Vertical, symbol Connector:Conn_01x02_Female
- removed J5: Bulb5, Connector_Molex:Molex_KK-254_AE-6410-02A_1x02_P2.54mm_Vertical, symbol Connector:Conn_01x02_Female
- removed J6: Bulb6, Connector_Molex:Molex_KK-254_AE-6410-02A_1x02_P2.54mm_Vertical, symbol Connector:Conn_01x02_Female
- removed J7: Bulb7, Connector_Molex:Molex_KK-254_AE-6410-02A_1x02_P2.54mm_Vertical, symbol Connector:Conn_01x02_Female
- removed J8: Bulb8, Connector_Molex:Molex_KK-254_AE-6410-02A_1x02_P2.54mm_Vertical, symbol Connector:Conn_01x02_Female
- removed K1, K2, K3, K4, K5, K6, K7, K8: SANYOU_SRD_Form_A, Relay_THT:Relay_SPST_SANYOU_SRD_Series_Form_A, symbol Relay:SANYOU_SRD_Form_A
- removed Q1, Q2, Q3, Q4, Q5, Q6, Q7, Q8: 2N3904, Package_TO_SOT_THT:TO-92_Inline, symbol Transistor_BJT:2N3904
- removed R1, R2, R3, R4, R5, R6, R7, R8: 1K, Resistor_THT:R_Axial_DIN0207_L6.3mm_D2.5mm_P10.16mm_Horizontal, symbol Device:R
- removed R10, R11, R12, R13, R14, R9: 4k7, Resistor_THT:R_Axial_DIN0207_L6.3mm_D2.5mm_P10.16mm_Horizontal, symbol Device:R
- removed U1, U2: 74HC4051, Package_DIP:DIP-16_W7.62mm, symbol 74xx:74HC4051
- removed XA1: Arduino_Nano_Socket, Arduino:Arduino_Nano_Socket, symbol AA-Arduino:Arduino_Nano_Socket
- added C1: 100nf, Capacitor_THT:C_Disc_D4.3mm_W1.9mm_P5.00mm, symbol Device:C
- added H1, H2, H3, H4: MountingHole_Pad, MountingHole:MountingHole_3.2mm_M3_DIN965_Pad, symbol Mechanical:MountingHole_Pad
- added J14: Reciver 10, Connector_PinSocket_2.54mm:PinSocket_1x07_P2.54mm_Vertical, symbol Connector:Conn_01x07_Female
- added J9: Reciver 9, Connector_PinSocket_2.54mm:PinSocket_1x07_P2.54mm_Vertical, symbol Connector:Conn_01x07_Female
- added XA1: Arduino_Mega2560_Pro_Mini, AA-ROB-FULL:MEGA2560PRO-EMBED, symbol AA-ROBSCH:Arduino_Mega2560_Pro_Mini
- J1: renamed from J9; footprint Connector_Molex:Molex_KK-254_AE-6410-05A_1x05_P2.54mm_Vertical -> Connector_PinHeader_2.54mm:PinHeader_1x10_P2.54mm_Vertical; symbol Connector:Conn_01x05_Female -> Connector:Conn_01x10_Female
- J2: renamed from J19; footprint Connector_PinSocket_2.54mm:PinSocket_1x11_P2.54mm_Vertical -> Connector_PinSocket_2.54mm:PinSocket_1x12_P2.54mm_Vertical; symbol Connector:Conn_01x11_Female -> Connector:Conn_01x12_Female
- renumbered C1 to C2, C2 to C3, D17 to D1, J14 to J10, J15 to J11, J16 to J12, J17 to J13, J20 to J3, J18 to J4, J10 to J5, J11 to J6, J12 to J7, J13 to J8, U3 to U1
Connections:
- net +5V: now also J3.4 (Pin_4), C1.2, J14.2 (Pin_2), J9.2 (Pin_2), XA1.5V1 (5V), XA1.5V2 (SPI_5V), XA1.5V3 (5V); no longer J3.3 (Pin_3)
- net GND: now also J1.10 (Pin_10), J2.12 (Pin_12), J3.3 (Pin_3), C1.1, H1.1, H2.1, H3.1, H4.1, J14.1 (Pin_1), J9.1 (Pin_1), XA1.GND1 (GND), XA1.GND2 (GND); no longer J1.5 (Pin_5), J2.11 (Pin_11), J3.4 (Pin_4)
- net Lamp1: now also XA1.D13
- net Lamp2: now also XA1.D22
- net Lamp3: now also XA1.D23
- net Lamp4: now also XA1.D24
- net Lamp5: now also XA1.D25
- net Lamp6: now also XA1.D26
- net Lamp7: now also XA1.D27
- net Lamp8: now also XA1.D28
- net Rec1: now also XA1.D44
- net Rec2: now also XA1.D45
- net Rec3: now also XA1.D46
- net Rec4: now also XA1.D47
- net Rec5: now also XA1.D48
- net Rec6: now also XA1.D49
- net Rec7: now also XA1.D50
- net Rec8: now also XA1.D51
- net SCL: now also XA1.D21 (D21_SCL)
- net SDA: now also XA1.D20 (D20_SDA)
- net at J2.3 (Pin_3): now also XA1.D4
- net at J2.4 (Pin_4): now also XA1.D5
- net at J2.5 (Pin_5): now also XA1.D6
- net at J2.6 (Pin_6): now also XA1.D7
- net at J2.10 (Pin_10): now also XA1.D11
- net at J2.9 (Pin_9): now also XA1.D10
- net Bonus: no longer names the net of J1.3 (Pin_3)
- net Bonus: now also XA1.D32
- net MP3-5: no longer names the net of J2.7 (Pin_7)
- net MP3-5: now also XA1.D8
- net MP3-6: no longer names the net of J2.8 (Pin_8)
- net MP3-6: now also XA1.D9
- net Reset: no longer names the net of J1.2 (Pin_2)
- net Reset: now also XA1.D31
- net Wrong: no longer names the net of J1.4 (Pin_4)
- net Wrong: now also XA1.D33
- new net: J2.11 (Pin_11), XA1.D12
- new net: J1.5 (Pin_5), XA1.D34
- new net: J1.6 (Pin_6), XA1.D35
- new net: J1.7 (Pin_7), XA1.D36
- new net: J1.8 (Pin_8), XA1.D37
- new net: J1.9 (Pin_9), XA1.D38
- new net Lamp10: XA1.D30
- new net Lamp9: XA1.D29
- new net Rec10: J14.6 (Pin_6), XA1.D53 (D53_SS)
- new net Rec9: J9.6 (Pin_6), XA1.D52
- no-connect marks 42 -> 43
Other:
- moved on the sheet: C2, C3, D1, J3, J4, U1
