File: HARDWARE/quizbuzzer/quizbuzzer.kicad_pcb (KiCad board)
At the start: 2 copper layers, 174 x 97.5 mm, 85 parts, among them J1 Controls, J10 Reciver 5, J11 Reciver 6, J12 Reciver 7, J13 Reciver 8, J14 Reciver 10, J15 Bulb1, J16 Bulb3, J17 Bulb3, J18 Bulb4, J19 Bulb5, J2 MP3out, J20 Bulb6, J21 Bulb7, J22 Bulb8, J23 Bulb9, J24 Bulb10, J3 I2C, J4 Powerjack, J5 Reciver 1, J6 Reciver 2, J7 Reciver 3, J8 Reciver 4, J9 Reciver 9, K1 SANYOU_SRD_Form_A, K10 SANYOU_SRD_Form_A, K2 SANYOU_SRD_Form_A, K3 SANYOU_SRD_Form_A, K4 SANYOU_SRD_Form_A, K5 SANYOU_SRD_Form_A, K6 SANYOU_SRD_Form_A, K7 SANYOU_SRD_Form_A, K8 SANYOU_SRD_Form_A, K9 SANYOU_SRD_Form_A, Q1 2N3904, Q10 2N3904, Q2 2N3904, Q3 2N3904, Q4 2N3904, Q5 2N3904, Q6 2N3904, Q7 2N3904, Q8 2N3904, Q9 2N3904, U1 L7805

Commit message: V0.1.1 Fixes
Parts:
- J3: footprint Connector_PinSocket_2.54mm:PinSocket_1x05_P2.54mm_Vertical -> Connector_PinSocket_2.54mm:PinSocket_1x04_P2.54mm_Vertical
- moved G*** 112.6 mm to (219.8, 48.0)
- moved J2 107.4 mm to (200.4, 72.0), turned to 270 degrees
- moved C1 69.4 mm to (40.9, 107.4), turned to 0 degrees
- moved C2 49.0 mm to (121.3, 99.9)
- moved C3 49.0 mm to (135.4, 99.9)
- moved D1 49.0 mm to (123.6, 103.5)
- moved J1 49.0 mm to (89.0, 108.4)
- moved J3 49.0 mm to (101.3, 102.5)
- moved J4 49.0 mm to (143.8, 99.2)
- moved U1 49.0 mm to (125.9, 109.2)
- moved J5 44.5 mm to (93.3, 69.9)
- moved J6 43.5 mm to (101.3, 69.9)
- moved J7 42.5 mm to (109.3, 69.9)
- moved J8 41.5 mm to (117.3, 69.9)
- moved J10 40.6 mm to (125.3, 69.9)
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Connections:
- J4 pad 1: GND -> +12V
- J4 pad 2: +12V -> GND
- J4 pad 3: (no net) -> GND
- J6 pad 1: Net-(J6-Pad1) -> GND
Routing:
- net GND: track 725.8 -> 0.00 mm
- net +5V: track 574.2 -> 0.00 mm
- net +12V: track 245.3 -> 0.00 mm
- net Rec9: track 172.9 -> 0.00 mm
- net Rec10: track 166.1 -> 0.00 mm
- net Lamp10: track 157.6 -> 0.00 mm
- net Rec7: track 151.5 -> 0.00 mm
- net Rec8: track 150.4 -> 0.00 mm
- net Lamp9: track 138.3 -> 0.00 mm
- net Rec6: track 136.5 -> 0.00 mm
- net Rec5: track 132.0 -> 0.00 mm
- net Rec4: track 131.5 -> 0.00 mm
- net Rec3: track 130.2 -> 0.00 mm
- net SDA: track 129.0 -> 0.00 mm
- net Net-(J1-Pad2): track 124.9 -> 0.00 mm, vias 1 -> 0
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- removed copper zone on F.Cu, net GND
Other:
- outline, holes or cut-outs redrawn
- board text added: "Quiz Buzzer V0.1.1 By TwinTurbo"
- board text removed: "Quiz Buzzer V0.1.0 By TwinTurbo"

Commit message: DMX and AuxConnector
Parts:
- removed G***: LOGO, AA-ROB-FULL:TOBINLOGO-BS
- added J25: Conn_02x12_Odd_Even, Connector_PinHeader_2.54mm:PinHeader_2x12_P2.54mm_Vertical, F.Cu at (51.6, 108.5)
- added J26: I2C, Connector_PinSocket_2.54mm:PinSocket_1x03_P2.54mm_Vertical, F.Cu at (160.4, 108.1)
- added U2: MAX485E, Package_DIP:DIP-8_W7.62mm_LongPads, F.Cu at (154.3, 92.3)
Connections:
- net Net-(XA1-PadD14) renamed AUX-HEAD-4
- net Net-(XA1-PadD15) renamed AUX-HEAD-3
- net Net-(XA1-PadD16) renamed AUX-HEAD-2
- net Net-(XA1-PadD17) renamed AUX-HEAD-1
- net Net-(XA1-PadD19) renamed DMX-RX
- J1 pad 2: Net-(J1-Pad2) -> Net-(J1-Pin_2)
- J1 pad 3: Net-(J1-Pad3) -> Net-(J1-Pin_3)
- J1 pad 4: Net-(J1-Pad4) -> Net-(J1-Pin_4)
- J1 pad 5: Net-(J1-Pad5) -> Net-(J1-Pin_5)
- J1 pad 6: Net-(J1-Pad6) -> Net-(J1-Pin_6)
- J1 pad 7: Net-(J1-Pad7) -> Net-(J1-Pin_7)
- J1 pad 8: Net-(J1-Pad8) -> Net-(J1-Pin_8)
- J1 pad 9: Net-(J1-Pad9) -> Net-(J1-Pin_9)
- J10 pad 3: Net-(J10-Pad3) -> unconnected-(J10-Pin_3-Pad3)
- J10 pad 4: Net-(J10-Pad4) -> unconnected-(J10-Pin_4-Pad4)
- J10 pad 5: Net-(J10-Pad5) -> unconnected-(J10-Pin_5-Pad5)
- J10 pad 7: Net-(J10-Pad7) -> unconnected-(J10-Pin_7-Pad7)
- J11 pad 3: Net-(J11-Pad3) -> unconnected-(J11-Pin_3-Pad3)
- J11 pad 4: Net-(J11-Pad4) -> unconnected-(J11-Pin_4-Pad4)
- J11 pad 5: Net-(J11-Pad5) -> unconnected-(J11-Pin_5-Pad5)
- J11 pad 7: Net-(J11-Pad7) -> unconnected-(J11-Pin_7-Pad7)
- J12 pad 3: Net-(J12-Pad3) -> unconnected-(J12-Pin_3-Pad3)
- J12 pad 4: Net-(J12-Pad4) -> unconnected-(J12-Pin_4-Pad4)
- J12 pad 5: Net-(J12-Pad5) -> unconnected-(J12-Pin_5-Pad5)
- J12 pad 7: Net-(J12-Pad7) -> unconnected-(J12-Pin_7-Pad7)
- J13 pad 3: Net-(J13-Pad3) -> unconnected-(J13-Pin_3-Pad3)
- J13 pad 4: Net-(J13-Pad4) -> unconnected-(J13-Pin_4-Pad4)
- J13 pad 5: Net-(J13-Pad5) -> unconnected-(J13-Pin_5-Pad5)
- J13 pad 7: Net-(J13-Pad7) -> unconnected-(J13-Pin_7-Pad7)
- J14 pad 3: Net-(J14-Pad3) -> unconnected-(J14-Pin_3-Pad3)
- J14 pad 4: Net-(J14-Pad4) -> unconnected-(J14-Pin_4-Pad4)
- J14 pad 5: Net-(J14-Pad5) -> unconnected-(J14-Pin_5-Pad5)
- J14 pad 7: Net-(J14-Pad7) -> unconnected-(J14-Pin_7-Pad7)
- J2 pad 10: Net-(J2-Pad10) -> Net-(J2-Pin_10)
- J2 pad 11: Net-(J2-Pad11) -> Net-(J2-Pin_11)
- J2 pad 3: Net-(J2-Pad3) -> Net-(J2-Pin_3)
- J2 pad 4: Net-(J2-Pad4) -> Net-(J2-Pin_4)
- J2 pad 5: Net-(J2-Pad5) -> Net-(J2-Pin_5)
- J2 pad 6: Net-(J2-Pad6) -> Net-(J2-Pin_6)
- J2 pad 7: Net-(J2-Pad7) -> Net-(J2-Pin_7)
- J2 pad 8: Net-(J2-Pad8) -> Net-(J2-Pin_8)
- J2 pad 9: Net-(J2-Pad9) -> Net-(J2-Pin_9)
- J3 pad 1: SCL -> +5V
- J3 pad 2: SDA -> GND
- J3 pad 3: GND -> SDA
- J3 pad 4: +5V -> SCL
- J5 pad 3: Net-(J5-Pad3) -> unconnected-(J5-Pin_3-Pad3)
- J5 pad 4: Net-(J5-Pad4) -> unconnected-(J5-Pin_4-Pad4)
- J5 pad 5: Net-(J5-Pad5) -> unconnected-(J5-Pin_5-Pad5)
- J5 pad 7: Net-(J5-Pad7) -> unconnected-(J5-Pin_7-Pad7)
- J6 pad 3: Net-(J6-Pad3) -> unconnected-(J6-Pin_3-Pad3)
- J6 pad 4: Net-(J6-Pad4) -> unconnected-(J6-Pin_4-Pad4)
- J6 pad 5: Net-(J6-Pad5) -> unconnected-(J6-Pin_5-Pad5)
- J6 pad 7: Net-(J6-Pad7) -> unconnected-(J6-Pin_7-Pad7)
- J7 pad 3: Net-(J7-Pad3) -> unconnected-(J7-Pin_3-Pad3)
- J7 pad 4: Net-(J7-Pad4) -> unconnected-(J7-Pin_4-Pad4)
- J7 pad 5: Net-(J7-Pad5) -> unconnected-(J7-Pin_5-Pad5)
- J7 pad 7: Net-(J7-Pad7) -> unconnected-(J7-Pin_7-Pad7)
- J8 pad 3: Net-(J8-Pad3) -> unconnected-(J8-Pin_3-Pad3)
- J8 pad 4: Net-(J8-Pad4) -> unconnected-(J8-Pin_4-Pad4)
- J8 pad 5: Net-(J8-Pad5) -> unconnected-(J8-Pin_5-Pad5)
- J8 pad 7: Net-(J8-Pad7) -> unconnected-(J8-Pin_7-Pad7)
- J9 pad 3: Net-(J9-Pad3) -> unconnected-(J9-Pin_3-Pad3)
- J9 pad 4: Net-(J9-Pad4) -> unconnected-(J9-Pin_4-Pad4)
- J9 pad 5: Net-(J9-Pad5) -> unconnected-(J9-Pin_5-Pad5)
- J9 pad 7: Net-(J9-Pad7) -> unconnected-(J9-Pin_7-Pad7)
- XA1 pad 3V3: Net-(XA1-Pad3V3) -> unconnected-(XA1-3.3V-Pad3V3)
- XA1 pad A0: Net-(XA1-PadA0) -> AUX-HEAD-5
- XA1 pad A1: Net-(XA1-PadA1) -> AUX-HEAD-6
- XA1 pad A10: Net-(XA1-PadA10) -> AUX-HEAD-15
- XA1 pad A11: Net-(XA1-PadA11) -> AUX-HEAD-16
- XA1 pad A12: Net-(XA1-PadA12) -> AUX-HEAD-17
- XA1 pad A13: Net-(XA1-PadA13) -> AUX-HEAD-18
- XA1 pad A14: Net-(XA1-PadA14) -> AUX-HEAD-19
- XA1 pad A15: Net-(XA1-PadA15) -> unconnected-(XA1-PadA15)
- XA1 pad A2: Net-(XA1-PadA2) -> AUX-HEAD-7
- XA1 pad A3: Net-(XA1-PadA3) -> AUX-HEAD-8
- XA1 pad A4: Net-(XA1-PadA4) -> AUX-HEAD-9
- XA1 pad A5: Net-(XA1-PadA5) -> AUX-HEAD-10
- XA1 pad A6: Net-(XA1-PadA6) -> AUX-HEAD-11
- XA1 pad A7: Net-(XA1-PadA7) -> AUX-HEAD-12
- XA1 pad A8: Net-(XA1-PadA8) -> AUX-HEAD-13
- XA1 pad A9: Net-(XA1-PadA9) -> AUX-HEAD-14
- XA1 pad AREF: Net-(XA1-PadAREF) -> unconnected-(XA1-PadAREF)
- XA1 pad D0: Net-(XA1-PadD0) -> unconnected-(XA1-D0_RX0-PadD0)
- XA1 pad D1: Net-(XA1-PadD1) -> unconnected-(XA1-D1_TX0-PadD1)
- XA1 pad D10: Net-(J2-Pad9) -> Net-(J2-Pin_11)
- XA1 pad D11: Net-(J2-Pad10) -> Lamp1
- XA1 pad D12: Net-(J2-Pad11) -> Lamp2
- XA1 pad D13: Lamp1 -> Lamp3
- XA1 pad D18: Net-(XA1-PadD18) -> DMX-TX
- XA1 pad D2: Net-(XA1-PadD2) -> Net-(J2-Pin_3)
- XA1 pad D22: Lamp2 -> Lamp4
- XA1 pad D23: Lamp3 -> Lamp5
- XA1 pad D24: Lamp4 -> Lamp6
- XA1 pad D25: Lamp5 -> Lamp7
- XA1 pad D26: Lamp6 -> Lamp8
- XA1 pad D27: Lamp7 -> Lamp9
- XA1 pad D28: Lamp8 -> Lamp10
- XA1 pad D29: Lamp9 -> Net-(J1-Pin_2)
- XA1 pad D3: Net-(XA1-PadD3) -> Net-(J2-Pin_4)
- XA1 pad D30: Lamp10 -> Net-(J1-Pin_3)
- XA1 pad D31: Net-(J1-Pad2) -> Net-(J1-Pin_4)
- XA1 pad D32: Net-(J1-Pad3) -> Net-(J1-Pin_5)
- XA1 pad D33: Net-(J1-Pad4) -> Net-(J1-Pin_6)
- XA1 pad D34: Net-(J1-Pad5) -> Net-(J1-Pin_7)
- XA1 pad D35: Net-(J1-Pad6) -> Net-(J1-Pin_8)
- XA1 pad D36: Net-(J1-Pad7) -> Net-(J1-Pin_9)
- XA1 pad D37: Net-(J1-Pad8) -> Rec1
- XA1 pad D38: Net-(J1-Pad9) -> Rec2
- XA1 pad D39: Net-(XA1-PadD39) -> Rec3
- XA1 pad D4: Net-(J2-Pad3) -> Net-(J2-Pin_5)
- XA1 pad D40: Net-(XA1-PadD40) -> Rec4
- XA1 pad D41: Net-(XA1-PadD41) -> Rec5
- XA1 pad D42: Net-(XA1-PadD42) -> Rec6
- XA1 pad D43: Net-(XA1-PadD43) -> Rec7
- XA1 pad D44: Rec1 -> Rec8
- XA1 pad D45: Rec2 -> Rec9
- XA1 pad D46: Rec3 -> Rec10
- XA1 pad D47: Rec4 -> AUX-HEAD-21
- XA1 pad D48: Rec5 -> AUX-HEAD-20
- XA1 pad D49: Rec6 -> AUX-HEAD-22
- XA1 pad D5: Net-(J2-Pad4) -> Net-(J2-Pin_6)
- XA1 pad D50: Rec7 -> AUX-HEAD-23
- XA1 pad D51: Rec8 -> AUX-HEAD-24
- XA1 pad D52: Rec9 -> AUX-HEAD-25
- XA1 pad D53: Rec10 -> AUX-HEAD-26
- XA1 pad D6: Net-(J2-Pad5) -> Net-(J2-Pin_7)
- XA1 pad D7: Net-(J2-Pad6) -> Net-(J2-Pin_8)
- XA1 pad D8: Net-(J2-Pad7) -> Net-(J2-Pin_9)
- XA1 pad D9: Net-(J2-Pad8) -> Net-(J2-Pin_10)
- XA1 pad GND3: (no net) -> GND
- XA1 pad MISO: Net-(XA1-PadMISO) -> unconnected-(XA1-SPI_MISO-PadMISO)
- XA1 pad MOSI: Net-(XA1-PadMOSI) -> unconnected-(XA1-SPI_MOSI-PadMOSI)
- XA1 pad RST: (no net) -> unconnected-(XA1-RESET-PadRST)
- XA1 pad RST1: Net-(XA1-PadRST1) -> unconnected-(XA1-RESET-PadRST1)
- XA1 pad SCK: Net-(XA1-PadSCK) -> unconnected-(XA1-SPI_SCK-PadSCK)
- XA1 pad VIN: Net-(XA1-PadVIN) -> unconnected-(XA1-PadVIN)
Other:
- net class Default removed
- board text added: "Quiz Buzzer V0.1.2 By TwinTurbo"
- board text removed: "Quiz Buzzer V0.1.1 By TwinTurbo"
