File: HARDWARE/quizbuzzer.kicad_pcb (KiCad board)
At the start: 2 copper layers, 174 x 97.5 mm, 87 parts, among them J1 Controls, J10 Reciver 5, J11 Reciver 6, J12 Reciver 7, J13 Reciver 8, J14 Reciver 10, J15 Bulb1, J16 Bulb3, J17 Bulb3, J18 Bulb4, J19 Bulb5, J2 MP3out, J20 Bulb6, J21 Bulb7, J22 Bulb8, J23 Bulb9, J24 Bulb10, J25 Conn_02x12_Odd_Even, J26 I2C, J3 I2C, J4 Powerjack, J5 Reciver 1, J6 Reciver 2, J7 Reciver 3, J8 Reciver 4, J9 Reciver 9, K1 SANYOU_SRD_Form_A, K10 SANYOU_SRD_Form_A, K2 SANYOU_SRD_Form_A, K3 SANYOU_SRD_Form_A, K4 SANYOU_SRD_Form_A, K5 SANYOU_SRD_Form_A, K6 SANYOU_SRD_Form_A, K7 SANYOU_SRD_Form_A, K8 SANYOU_SRD_Form_A, K9 SANYOU_SRD_Form_A, Q1 2N3904, Q10 2N3904, Q2 2N3904, Q3 2N3904, Q4 2N3904, Q5 2N3904, Q6 2N3904, Q7 2N3904, Q8 2N3904, Q9 2N3904, U1 L7805, U2 MAX485E

Commit message: FIXLAYER
Parts:
- J25: value Conn_02x12_Odd_Even -> Conn_02x14_Odd_Even; footprint Connector_PinHeader_2.54mm:PinHeader_2x12_P2.54mm_Vertical -> Connector_PinHeader_2.54mm:PinHeader_2x14_P2.54mm_Vertical
- J26: value I2C -> DMX
Connections:
- J2 pad 10: Net-(J2-Pin_10) -> PORTB_8
- J2 pad 11: Net-(J2-Pin_11) -> MP3_EN
- J2 pad 3: Net-(J2-Pin_3) -> PORTB_1
- J2 pad 4: Net-(J2-Pin_4) -> PORTB_2
- J2 pad 5: Net-(J2-Pin_5) -> PORTB_3
- J2 pad 6: Net-(J2-Pin_6) -> PORTB_4
- J2 pad 7: Net-(J2-Pin_7) -> PORTB_5
- J2 pad 8: Net-(J2-Pin_8) -> PORTB_6
- J2 pad 9: Net-(J2-Pin_9) -> PORTB_7
- J25 pad 1: AUX-HEAD-5 -> AUX-HEAD-1
- J25 pad 10: AUX-HEAD-21 -> AUX-HEAD-18
- J25 pad 11: AUX-HEAD-10 -> AUX-HEAD-6
- J25 pad 12: AUX-HEAD-20 -> AUX-HEAD-19
- J25 pad 13: AUX-HEAD-11 -> AUX-HEAD-7
- J25 pad 14: AUX-HEAD-22 -> AUX-HEAD-21
- J25 pad 15: AUX-HEAD-12 -> AUX-HEAD-8
- J25 pad 16: AUX-HEAD-23 -> AUX-HEAD-20
- J25 pad 17: AUX-HEAD-13 -> AUX-HEAD-9
- J25 pad 18: AUX-HEAD-24 -> AUX-HEAD-22
- J25 pad 19: AUX-HEAD-14 -> AUX-HEAD-10
- J25 pad 2: AUX-HEAD-16 -> AUX-HEAD-14
- J25 pad 20: AUX-HEAD-25 -> AUX-HEAD-23
- J25 pad 21: AUX-HEAD-15 -> AUX-HEAD-11
- J25 pad 22: AUX-HEAD-26 -> AUX-HEAD-24
- J25 pad 23: GND -> AUX-HEAD-12
- J25 pad 24: +5V -> AUX-HEAD-25
- J25 pad 3: AUX-HEAD-6 -> AUX-HEAD-2
- J25 pad 4: AUX-HEAD-17 -> AUX-HEAD-15
- J25 pad 5: AUX-HEAD-7 -> AUX-HEAD-3
- J25 pad 6: AUX-HEAD-18 -> AUX-HEAD-16
- J25 pad 7: AUX-HEAD-8 -> AUX-HEAD-4
- J25 pad 8: AUX-HEAD-19 -> AUX-HEAD-17
- J25 pad 9: AUX-HEAD-9 -> AUX-HEAD-5
- XA1 pad A15: unconnected-(XA1-PadA15) -> AUX-HEAD-20
- XA1 pad D10: Net-(J2-Pin_11) -> AUX-HEAD-27
- XA1 pad D2: Net-(J2-Pin_3) -> MP3_EN
- XA1 pad D3: Net-(J2-Pin_4) -> AUX-HEAD-24
- XA1 pad D4: Net-(J2-Pin_5) -> PORTB_1
- XA1 pad D48: AUX-HEAD-20 -> AUX-HEAD-22
- XA1 pad D49: AUX-HEAD-22 -> AUX-HEAD-23
- XA1 pad D5: Net-(J2-Pin_6) -> PORTB_2
- XA1 pad D50: AUX-HEAD-23 -> PORTB_5
- XA1 pad D51: AUX-HEAD-24 -> PORTB_6
- XA1 pad D52: AUX-HEAD-25 -> PORTB_7
- XA1 pad D53: AUX-HEAD-26 -> PORTB_8
- XA1 pad D6: Net-(J2-Pin_7) -> PORTB_3
- XA1 pad D7: Net-(J2-Pin_8) -> PORTB_4
- XA1 pad D8: Net-(J2-Pin_9) -> AUX-HEAD-25
- XA1 pad D9: Net-(J2-Pin_10) -> AUX-HEAD-26
Routing:
- net GND: track 0.00 -> 773.5 mm
- net +5V: track 0.00 -> 630.4 mm
- net +12V: track 0.00 -> 245.1 mm
- net PORTB_1: track 0.00 -> 154.9 mm
- net PORTB_4: track 0.00 -> 153.5 mm
- net PORTB_2: track 0.00 -> 152.4 mm
- net MP3_EN: track 0.00 -> 149.5 mm
- net PORTB_3: track 0.00 -> 145.8 mm
- net Lamp10: track 0.00 -> 136.3 mm
- net Lamp9: track 0.00 -> 119.4 mm, vias 0 -> 1
- net PORTB_5: track 0.00 -> 113.4 mm
- net Lamp8: track 0.00 -> 104.7 mm, vias 0 -> 1
- net AUX-HEAD-22: track 0.00 -> 104.6 mm, vias 0 -> 1
- net AUX-HEAD-23: track 0.00 -> 103.2 mm
- net PORTB_6: track 0.00 -> 102.3 mm
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