File: HARDWARE/quizbuzzer.sch (KiCad schematic (older format))
At the start: 24 parts, among them J1 Controls, J10 Reciver 5, J11 Reciver 6, J12 Reciver 7, J13 Reciver 8, J14 Reciver 10, J2 MP3out, J3 I2C, J4 Powerjack, J5 Reciver 1, J6 Reciver 2, J7 Reciver 3, J8 Reciver 4, J9 Reciver 9, U1 L7805

Commit message: Fixing Corrupt
Parts:
- added J25: Conn_02x12_Odd_Even, symbol Connector_Generic:Conn_02x12_Odd_Even
- added J26: I2C, Connector_PinSocket_2.54mm:PinSocket_1x03_P2.54mm_Vertical, symbol Connector:Conn_01x03_Pin
- added U2: MAX485E, symbol Interface_UART:MAX485E
- J1: symbol Connector:Conn_01x10_Female -> quizbuzzer-rescue:Conn_01x10_Female-Connector
- J10, J11, J12, J13, J14, J5, J6, J7, J8, J9: symbol Connector:Conn_01x07_Female -> quizbuzzer-rescue:Conn_01x07_Female-Connector
- J2: symbol Connector:Conn_01x12_Female -> quizbuzzer-rescue:Conn_01x12_Female-Connector
- J3: symbol Connector:Conn_01x04_Female -> quizbuzzer-rescue:Conn_01x04_Female-Connector
- XA1: symbol AA-ROBSCH:Arduino_Mega2560_Pro_Mini -> quizbuzzer-rescue:Arduino_Mega2560_Pro_Mini-AA-ROBSCH
Connections:
- net labels added: AUX-HEAD-1, AUX-HEAD-10, AUX-HEAD-11, AUX-HEAD-12, AUX-HEAD-13, AUX-HEAD-14, AUX-HEAD-15, AUX-HEAD-16, AUX-HEAD-17, AUX-HEAD-18, AUX-HEAD-19, AUX-HEAD-2, AUX-HEAD-20, AUX-HEAD-21, AUX-HEAD-22, AUX-HEAD-23, AUX-HEAD-24, AUX-HEAD-25, AUX-HEAD-26, AUX-HEAD-3, AUX-HEAD-4, AUX-HEAD-5, AUX-HEAD-6, AUX-HEAD-7, AUX-HEAD-8, AUX-HEAD-9, DMX-RX, DMX-TX
- wire segments 46 -> 48
- no-connect marks 42 -> 46
Other:
- moved on the sheet: H1, H2, H3, H4
